File: Electric/Aeris control electrical plans/Aeris control electrical plans.kicad_sch (KiCad schematic)
At the start: 6 parts, among them J1 Battery barrel jack, J2 Electrical barrel jack, M1 Stepper_Motor_bipolar, U1 Pico, U2 A4988_STEPPER_MOTOR_DRIVER_CA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

Commit message: push élec presque terminé
Parts:
- added J3: Conn_+5V, symbol Connector:Conn_01x02_Pin
- added J4, J7: Conn_+3v3, symbol Connector:Conn_01x02_Pin
- added J5, J6: Conn_+12V, symbol Connector:Conn_01x02_Pin
- added M2: Stepper_Motor_bipolar, symbol Motor:Stepper_Motor_bipolar
- added U3: A4988_DRIVER_CARRIER, A4988_STEPPER_MOTOR_DRIVER_CARRIER:MODULE_A4988_STEPPER_MOTOR_DRIVER_CARRIER, symbol A4988:A4988_STEPPER_MOTOR_DRIVER_CARRIER
- added U4, U5: LM2596_module, symbol Buck_converter_modules:LM2596_Module
- J1: value Battery barrel jack -> Battery barrel jack 12V
- J2: value Electrical barrel jack -> Electrical barrel jack 12V
- U2: value A4988_STEPPER_MOTOR_DRIVER_CARRIER -> A4988_DRIVER_CARRIER
Connections:
- net +12V: now also J2.1, U2.16 (VMOT), J5.1 (Pin_1), J6.1 (Pin_1), U3.16 (VMOT), U4.1 (In+), U5.1 (In+)
- net GND: now also J2.2, U1.13 (GND), U1.18 (GND), U1.23 (GND), U1.28 (GND), U1.3 (GND), U1.33 (AGND), U1.38 (GND), U1.42 (GND), U1.8 (GND), U2.15 (GND), U2.9 (GND), J3.2 (Pin_2), J4.2 (Pin_2), J5.2 (Pin_2), J6.2 (Pin_2), J7.2 (Pin_2), U3.15 (GND), U3.9 (GND), U4.2 (In-), U4.4 (Out-), U5.2 (In-), U5.4 (Out-)
- net +3V3: now reaches U2.10 (VDD)
- net +3V3: now also U1.39 (VSYS), J4.1 (Pin_1), J7.1 (Pin_1), U3.10 (VDD), U5.3 (Out+)
- net at U2.11 (1B): now also M1.1
- net at U2.12 (1A): now also M1.2 (-)
- net at U2.13 (2A): now also M1.3
- net at U2.14 (2B): now also M1.4
- net at U2.5 (~{RESET}): now also U2.6 (~{SLEEP})
- new net: M2.1, U3.11 (1B)
- new net: M2.2 (-), U3.12 (1A)
- new net: M2.3, U3.13 (2A)
- new net: M2.4, U3.14 (2B)
- new net: U3.5 (~{RESET}), U3.6 (~{SLEEP})
- new net +5V: J3.1 (Pin_1), U4.3 (Out+)
- no-connect marks 0 -> 11
Other:
- note added: "+3V3"
- note added: "+5V"
- note added: "Buck converters modules"
- moved on the sheet: J1, J2, M1, U1, U2

Commit message: Push motor code
Parts:
- added J8, J9: Conn_Pico_1, symbol Connector:Conn_01x02_Pin
Connections:
- net at U2.7 (STEP): now also J8.1 (Pin_1)
- net at U2.8 (DIR): now also J8.2 (Pin_2)
- net at U3.7 (STEP): now also J9.1 (Pin_1)
- net at U3.8 (DIR): now also J9.2 (Pin_2)
Other:
- note added: "Pico to stepper driver dev board"

Commit message: Push schéma électrique + pdf
Parts:
- added J10: Conn_Pico_3, symbol Connector:Conn_01x02_Pin
- added J11: Conn_Alim, symbol Connector:Conn_01x03_Pin
- added J12: Conn_Motor_Z, symbol Connector:Conn_01x02_Pin
- added J13: Conn_Motor_PORT, symbol Connector:Conn_01x02_Pin
- added J14: Conn_Motor_STARBOARD, symbol Connector:Conn_01x02_Pin
- added J15: Conn_UART, symbol Connector:Conn_01x04_Pin
- added J16: Conn_I2C_IMU_MAST, symbol Connector:Conn_01x04_Pin
- added J17: Conn_I2C_IMU_PLANK, symbol Connector:Conn_01x04_Pin
- added J18: Conn_I2C_ANEMOMETER, symbol Connector:Conn_01x04_Pin
- added J19: Conn_I2C_VANE, symbol Connector:Conn_01x04_Pin
- added J20: Conn_+3v3, symbol Connector:Conn_01x02_Pin
- added J21: Conn_+3v3_1M_Board, symbol Connector:Conn_01x02_Pin
- added J22: Conn_+3v3_2M_Board, symbol Connector:Conn_01x02_Pin
- added M3: Stepper_Motor_bipolar, symbol Motor:Stepper_Motor_bipolar
- added U6: A4988_DRIVER_CARRIER, A4988_STEPPER_MOTOR_DRIVER_CARRIER:MODULE_A4988_STEPPER_MOTOR_DRIVER_CARRIER, symbol A4988:A4988_STEPPER_MOTOR_DRIVER_CARRIER
- J9: value Conn_Pico_1 -> Conn_Pico_2
Connections:
- net +12V: now also J11.1 (Pin_1), U6.16 (VMOT)
- net +3V3: now also J11.2 (Pin_2), J16.1 (Pin_1), J17.1 (Pin_1), J18.1 (Pin_1), J19.1 (Pin_1), J20.1 (Pin_1), J21.1 (Pin_1), J22.1 (Pin_1), U6.10 (VDD)
- net GND: now also J11.3 (Pin_3), J15.4 (Pin_4), J16.4 (Pin_4), J17.4 (Pin_4), J18.4 (Pin_4), J19.4 (Pin_4), J20.2 (Pin_2), J21.2 (Pin_2), J22.2 (Pin_2), U6.15 (GND), U6.9 (GND)
- net UART_TX: now reaches U1.1 (GPIO0)
- net UART_TX: now also J15.2 (Pin_2)
- net STEP_Z: now reaches U1.19 (GPIO14)
- net STEP_Z: now also J12.1 (Pin_1)
- net UART_RX: now reaches U1.2 (GPIO1)
- net UART_RX: now also J15.3 (Pin_3)
- net DIR_Z: now reaches U1.20 (GPIO15)
- net DIR_Z: now also J12.2 (Pin_2)
- net DIR_PORT: now reaches U1.21 (GPIO16)
- net DIR_PORT: now also J13.2 (Pin_2)
- net STEP_PORT: now reaches U1.22 (GPIO17)
- net STEP_PORT: now also J13.1 (Pin_1)
- net DIR_STAR: now reaches U1.24 (GPIO18)
- net DIR_STAR: now also J14.2 (Pin_2)
- net STEP_STAR: now reaches U1.25 (GPIO19)
- net STEP_STAR: now also J14.1 (Pin_1)
- net I2C_SDA: now reaches U1.6 (GPIO4)
- net I2C_SDA: now also J16.2 (Pin_2), J17.2 (Pin_2), J18.2 (Pin_2), J19.2 (Pin_2)
- net I2C_SCL: now reaches U1.7 (GPIO5)
- net I2C_SCL: now also J16.3 (Pin_3), J17.3 (Pin_3), J18.3 (Pin_3), J19.3 (Pin_3)
- new net: M3.1, U6.11 (1B)
- new net: M3.2 (-), U6.12 (1A)
- new net: M3.3, U6.13 (2A)
- new net: M3.4, U6.14 (2B)
- new net: U6.5 (~{RESET}), U6.6 (~{SLEEP})
- new net: J10.1 (Pin_1), U6.7 (STEP)
- new net: J10.2 (Pin_2), U6.8 (DIR)
- no-connect marks 11 -> 36
Other:
- note added: "Pico to one stepper driver dev board"
- note added: "Pico to two stepper driver dev board"
- note added: "Protoboard for the Rpico RP2350 This board is mostly made out of connectors so the RP2350 may communicate with different modules. It is also used to redistribute 3v3 and GND to all of the other modules."
- note removed: "Pico to stepper driver dev board"
- company: (none) -> Université de Sherbrooke
- title: (none) -> Aeris control electrical schematic
- moved on the sheet: J6, J7, J8, J9, M1, M2, U1, U2, U3
