File: Electric/Aeris control electrical plans/Cerbrum_Aeris/Cerbrum_Aeris.kicad_sch (KiCad schematic)
At the start: 0 parts

Commit message: push éelectrique pcb
Other:
- sheet MCU ports: added GPIO[0..1], GPIO[2..3], GPIO[4..5]; removed GPIO[0..2], GPIO[3..5]
- sheet RPi connection ports: added GPIO[0..1]; removed none
- sheet Sensors ports: added GPIO[2..3]; removed none
- note added: "I2C_0"
- note added: "I2C_1"
- note added: "M_Conn_LEFT"
- note added: "M_Conn_RIGHT"
- note added: "UART"
- note added: "Unused"
Changed lines of the file:
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@@
 	(generator_version "9.0")
 	(paper "A4")
+	(text "Unused"
+		(exclude_from_sim no)
+		(at 68.834 57.404 0)
+		(effects
+			(font
+				(size 1.27 1.27)
+				(thickness 0.254)
+				(bold yes)
+			)
+		)
+	)
+	(text "I2C_1"
+		(exclude_from_sim no)
+		(at 71.374 32.004 0)
+		(effects
+			(font
+				(size 1.27 1.27)
+				(thickness 0.254)
+				(bold yes)
+			)
+		)
+	)
+	(text "M_Conn_RIGHT"
+		(exclude_from_sim no)
+		(at 65.532 52.07 0)
+		(effects
+			(font
+				(size 1.27 1.27)
+				(thickness 0.254)
+				(bold yes)
+			)
+		)
+	)
+	(text "I2C_0"
+		(exclude_from_sim no)
+		(at 71.882 29.21 0)
+		(effects
+			(font
+				(size 1.27 1.27)
+				(thickness 0.254)
+				(bold yes)
+			)
+		)
+	)
+	(text "UART"
+		(exclude_from_sim no)
+		(at 72.644 39.116 0)
+		(effects
+			(font
+				(size 1.27 1.27)
+				(thickness 0.254)
+				(bold yes)
+			)
+		)
+	)
+	(text "M_Conn_LEFT"
+		(exclude_from_sim no)
+		(at 67.056 46.99 0)
+		(effects
+			(font
+				(size 1.27 1.27)
+				(thickness 0.254)
+				(bold yes)
+			)
+		)
+	)
 	(no_connect
 		(at 86.36 57.15)
@@
 	(bus
 		(pts
+			(xy 101.6 87.63) (xy 134.62 87.63)
+		)
+		(stroke
+			(width 0)
+			(type default)
+		)
+	)
+	(bus
+		(pts
 			(xy 96.52 46.99) (xy 86.36 46.99)
 		)
@@
 	(bus
 		(pts
+			(xy 104.14 31.75) (xy 104.14 39.37)
+		)
+		(stroke
+			(width 0)
+			(type default)
+		)
+	)
+	(bus
+		(pts
 			(xy 106.68 29.21) (xy 86.36 29.21)
 		)
@@
 	(bus
 		(pts
+			(xy 101.6 39.37) (xy 101.6 87.63)
+		)
+		(stroke
+			(width 0)
+			(type default)
+		)
+	)
+	(bus
+		(pts
 			(xy 86.36 120.65) (xy 88.9 120.65)
 		)
@@
 		(pts
 			(xy 134.62 36.83) (xy 106.68 36.83)
+		)
+		(stroke
+			(width 0)
+			(type default)
+		)
+	)
+	(bus
+		(pts
+			(xy 86.36 39.37) (xy 101.6 39.37)
+		)
+		(stroke
+			(width 0)
+			(type default)
+		)
+	)
+	(bus
+		(pts
+			(xy 86.36 31.75) (xy 104.14 31.75)
+		)
+		(stroke
+			(width 0)
+			(type default)
+		)
+	)
+	(bus
+		(pts
+			(xy 104.14 39.37) (xy 134.62 39.37)
 		)
 		(stroke
@@
 			)
 		)
+		(pin "GPIO[2..3]" input
+			(at 134.62 39.37 180)
+			(effects
+				(font
+					(size 1.27 1.27)
+				)
+				(justify left)
+			)
+		)
 		(instances
 			(project "Cerbrum_Aeris"
@@
 			)
 		)
-		(pin "GPIO[0..2]" input
-			(at 86.36 39.37 0)
-			(effects
-				(font
-					(size 1.27 1.27)
-				)
-				(justify right)
-			)
-		)
-		(pin "GPIO[3..5]" input
+		(pin "GPIO[4..5]" input
 			(at 86.36 29.21 0)
 			(effects
@@
 		(pin "GPIO[24..47]" input
 			(at 86.36 57.15 0)
+			(effects
+				(font
+					(size 1.27 1.27)
+				)
+				(justify right)
+			)
+		)
+		(pin "GPIO[0..1]" input
+			(at 86.36 39.37 0)
+			(effects
+				(font
+					(size 1.27 1.27)
+				)
+				(justify right)
+			)
+		)
+		(pin "GPIO[2..3]" input
+			(at 86.36 31.75 0)
 			(effects
 				(font
@@
 			)
 		)
+		(pin "GPIO[0..1]" input
+			(at 134.62 87.63 180)
+			(effects
+				(font
+					(size 1.27 1.27)
+				)
+				(justify left)
+			)
+		)
