File: Electric/Aeris control electrical plans/Cerbrum_Aeris/Power.kicad_sch (KiCad schematic)
At the start: 25 parts, among them Q1 AO3401A, U4 AP7361C-33E

Commit message: push éelectrique pcb
Parts:
- added J31: ~, Custom_Aeris:SJ_Stepper_1-5mm, symbol Aeris_custom:SJ_Stepper_1-5mm
- BT1: footprint (none) -> TerminalBlock:TerminalBlock_Altech_AK300-2_P5.00mm
Connections:
- net +12V: now also J31.2 (b); no longer BT1.1 (+), C20.1, C21.1, R9.1, TP2.1, U6.1 (VIN)
- net GND: now also J31.1 (a), J31.4 (d); no longer BT1.2 (-), C20.2, C21.2, C25.2, C26.2, R10.2, R13.2, TP5.1, U6.3 (GND), U6.4 (AGND)
- net VIN_PROTECTION renamed +5V_ALIM
- net +5V_ALIM: now also J31.6 (C); no longer C19.2, FB1.2, TP1.1, U4.1 (VI)
- net Vcc_3V3 renamed +3V3
- new net +12V_BAT: BT1.1 (+), C20.1, C21.1, J31.7 (B), R9.1, TP2.1, U6.1 (VIN)
- new net +5V: C19.2, FB1.2, J31.3 (c), TP1.1, U4.1 (VI)
- new net GND_ALIM: BT1.2 (-), C20.2, C21.2, C25.2, C26.2, J31.5 (D), J31.8 (A), R10.2, R13.2, TP5.1, U6.3 (GND), U6.4 (AGND)
Other:
- note added: "3Amps traces"
- moved on the sheet: C19, C22, D1, R11, TP3, TP4, U4
