File: Electric/Aeris control electrical plans/Cerbrum_Aeris/Sensors.kicad_sch (KiCad schematic)
At the start: 6 parts, among them J15 Conn_01x04_Socket, J16 Conn_01x04_Socket, J17 Conn_01x04_Socket, J18 Conn_01x04_Socket

Commit message: push éelectrique pcb
Parts:
- removed J17, J18: Conn_01x04_Socket, symbol Connector:Conn_01x04_Socket
- added J19, J21, J23, J24, J27, J29: Conn_01x04_Socket, Connector_PinSocket_2.54mm:PinSocket_1x04_P2.54mm_Vertical, symbol Connector:Conn_01x04_Socket
- added J28, J30: ~, Custom_Aeris:SJ_Stepper_1-5mm, symbol Aeris_custom:SJ_Stepper_1-5mm
- added R20, R21: 10k, Resistor_SMD:R_0603_1608Metric, symbol Device:R_US
- J15, J16: footprint (none) -> Connector_PinSocket_2.54mm:PinSocket_1x04_P2.54mm_Vertical
- R18, R19: footprint (none) -> Resistor_SMD:R_0603_1608Metric
Connections:
- net +3V3: now also J28.1 (a), J30.1 (a), R20.1, R21.1; no longer J15.1 (Pin_1), J16.1 (Pin_1)
- net GND: now also J28.4 (d), J30.4 (d); no longer J15.4 (Pin_4), J16.4 (Pin_4)
- net GPIO4: now also J28.2 (b); no longer J15.2 (Pin_2), J16.2 (Pin_2)
- net GPIO5: now also J28.3 (c); no longer J15.3 (Pin_3), J16.3 (Pin_3)
- new net +3V3_I2C: J15.1 (Pin_1), J16.1 (Pin_1), J19.1 (Pin_1), J21.1 (Pin_1), J23.1 (Pin_1), J24.1 (Pin_1), J27.1 (Pin_1), J28.8 (A), J29.1 (Pin_1), J30.8 (A)
- new net GND_I2C: J15.4 (Pin_4), J16.4 (Pin_4), J19.4 (Pin_4), J21.4 (Pin_4), J23.4 (Pin_4), J24.4 (Pin_4), J27.4 (Pin_4), J28.5 (D), J29.4 (Pin_4), J30.5 (D)
- new net GPIO2: J30.2 (b), R20.2
- new net GPIO3: J30.3 (c), R21.2
- new net SCL_0: J15.3 (Pin_3), J16.3 (Pin_3), J19.3 (Pin_3), J21.3 (Pin_3), J28.6 (C)
- new net SCL_1: J23.3 (Pin_3), J24.3 (Pin_3), J27.3 (Pin_3), J29.3 (Pin_3), J30.6 (C)
- new net SDA_0: J15.2 (Pin_2), J16.2 (Pin_2), J19.2 (Pin_2), J21.2 (Pin_2), J28.7 (B)
- new net SDA_1: J23.2 (Pin_2), J24.2 (Pin_2), J27.2 (Pin_2), J29.2 (Pin_2), J30.7 (B)
Other:
- moved on the sheet: R18, R19
