File: Electric/Aeris control electrical plans/Cerbrum_Aeris/Cerbrum_Aeris.kicad_pcb (KiCad board)
At the start: 2 copper layers, 77 parts, among them J1 USB_C_PICO, J10 Conn_01x08_Stepper, J11 Conn_09x16_Stepper, J12 Conn_09x16_Stepper, J13 Conn_09x16_Stepper, J14 Raspberry_Pi_4, J2 Conn_01x08_Stepper, J3 Conn_01x08_Stepper, J4 Conn_01x08_Stepper, J5 Conn_09x16_Stepper, J6 Conn_09x16_Stepper, J7 Conn_09x16_Stepper, J8 Conn_01x08_Stepper, J9 Conn_01x08_Stepper, M1 Stepper_Motor_bipolar, M2 Stepper_Motor_bipolar, M3 Stepper_Motor_bipolar, M4 Stepper_Motor_bipolar, M5 Stepper_Motor_bipolar, M6 Stepper_Motor_bipolar, Q1 AO3401A, SW1 SW_BOOTSEL, SW2 SW_RESET, U1 SRV05-4, U2 RP2350B-QFN80, U3 W25Q128JVPIQ, U4 AP7361C-33E, U5 TPS562242DRLR, Y1 CM4012M00012001

Commit message: push éelectrique pcb
Parts:
- removed C23: 0.1µF, Capacitor_SMD:C_0603_1608Metric_Pad1.08x0.95mm_HandSolder
- removed U5: TPS562242DRLR, Package_TO_SOT_SMD:SOT-563
- added BT1: Battery, TerminalBlock:TerminalBlock_Altech_AK300-2_P5.00mm, B.Cu at (219.8, 99.3)
- added H2: MountingHole, MountingHole:MountingHole_3.5mm, F.Cu at (147.5, 121.0)
- added H4: MountingHole, MountingHole:MountingHole_3.5mm, F.Cu at (204.5, 121.0)
- added J15: Conn_01x04_Socket, Connector_PinSocket_2.54mm:PinSocket_1x04_P2.54mm_Vertical, B.Cu at (128.5, 73.9)
- added J16: Conn_01x04_Socket, Connector_PinSocket_2.54mm:PinSocket_1x04_P2.54mm_Vertical, B.Cu at (128.5, 79.4)
- added J17: ~, Custom_Aeris:SJ_Stepper_1-5mm, F.Cu at (153.2, 67.8)
- added J18: ~, Custom_Aeris:SJ_Stepper_1-5mm, F.Cu at (173.8, 67.8)
- added J19: Conn_01x04_Socket, Connector_PinSocket_2.54mm:PinSocket_1x04_P2.54mm_Vertical, B.Cu at (128.5, 85.0)
- added J20: ~, Custom_Aeris:SJ_Stepper_1-5mm, F.Cu at (194.2, 67.8)
- added J21: Conn_01x04_Socket, Connector_PinSocket_2.54mm:PinSocket_1x04_P2.54mm_Vertical, B.Cu at (128.5, 90.6)
- added J22: ~, Custom_Aeris:SJ_Stepper_1-5mm, F.Cu at (157.8, 125.2)
- added J23: Conn_01x04_Socket, Connector_PinSocket_2.54mm:PinSocket_1x04_P2.54mm_Vertical, B.Cu at (128.5, 102.5)
- added J24: Conn_01x04_Socket, Connector_PinSocket_2.54mm:PinSocket_1x04_P2.54mm_Vertical, B.Cu at (128.5, 108.1)
- added J25: ~, Custom_Aeris:SJ_Stepper_1-5mm, F.Cu at (178.2, 125.2)
- added J26: ~, Custom_Aeris:SJ_Stepper_1-5mm, F.Cu at (198.8, 125.2)
- added J27: Conn_01x04_Socket, Connector_PinSocket_2.54mm:PinSocket_1x04_P2.54mm_Vertical, B.Cu at (128.5, 113.7)
- added J28: ~, Custom_Aeris:SJ_Stepper_1-5mm, F.Cu at (143.2, 81.8)
- added J29: Conn_01x04_Socket, Connector_PinSocket_2.54mm:PinSocket_1x04_P2.54mm_Vertical, B.Cu at (128.5, 119.5)
- added J30: ~, Custom_Aeris:SJ_Stepper_1-5mm, F.Cu at (143.2, 116.0)
- added J31: ~, Custom_Aeris:SJ_Stepper_1-5mm, F.Cu at (208.8, 94.2)
- added L1: 3.3uH, Resistor_SMD:R_0805_2012Metric, B.Cu at (173.7, 88.6)
- added R18: 10k, Resistor_SMD:R_0603_1608Metric, B.Cu at (150.3, 80.3)
- added R19: 10k, Resistor_SMD:R_0603_1608Metric, B.Cu at (150.3, 78.7)
- added R20: 10k, Resistor_SMD:R_0603_1608Metric, B.Cu at (150.4, 114.5)
- added R21: 10k, Resistor_SMD:R_0603_1608Metric, B.Cu at (150.4, 113.0)
- added U6: ~, Package_TO_SOT_SMD:SOT-563, F.Cu at (218.0, 111.6)
- C1, C10, C11, C12, C13, C14, C15, C16, C17, C18, C19, C2, C22, C3, C4, C5, C6, C7, C8, C9, F1, FB1, J1, J14, M1, M2, M3, M4, M5, M6, Q1, R11, R3, R4, R5, R6, R7, R8, U1, U2, U3, U4, Y1: moved to B.Cu
- L2: value 3,3µH 40mOhm -> 2.2uH 13.2mOhm; moved to B.Cu
- R10: value 32k -> 17.4k
- R12: value 154k -> 220k
- TP2, TP4: footprint TestPoint:TestPoint_Pad_D1.0mm -> TestPoint:TestPoint_Pad_D4.0mm; moved to B.Cu
- TP5: footprint TestPoint:TestPoint_Pad_1.0x1.0mm -> TestPoint:TestPoint_Pad_4.0x4.0mm; moved to B.Cu
- moved M4 169.0 mm to (196.5, 140.3)
- moved M3 167.8 mm to (196.5, 53.2), turned to 180 degrees
- moved J14 159.8 mm to (176.5, 72.0), turned to -90 degrees
- moved R9 159.0 mm to (224.0, 106.9), turned to -90 degrees
- moved TP4 157.6 mm to (222.7, 71.8), turned to 180 degrees
- moved R10 156.5 mm to (221.5, 107.8), turned to 180 degrees
- moved R13 153.5 mm to (218.1, 107.8)
- moved M2 152.2 mm to (176.0, 53.2), turned to 180 degrees
- moved TP5 152.2 mm to (217.7, 77.5), turned to 180 degrees
- moved R12 149.9 mm to (214.7, 107.8)
- moved C24 149.8 mm to (214.7, 109.3)
- moved C26 147.7 mm to (212.5, 98.2), turned to -90 degrees
- moved C21 147.5 mm to (212.5, 94.8), turned to 90 degrees
- moved TP2 146.7 mm to (212.8, 71.8), turned to 180 degrees
- moved C4 145.7 mm to (184.1, 94.3)
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Connections:
- C19 pad 2: VIN_PROTECTION -> +5V
- C20 pad 1: +12V -> +12V_BAT
- C20 pad 2: GND -> GND_ALIM
- C21 pad 1: +12V -> +12V_BAT
- C21 pad 2: GND -> GND_ALIM
- C22 pad 2: Vcc_3V3 -> +3V3
- C24 pad 1: VIN_PROTECTION -> +5V_ALIM
- C25 pad 1: VIN_PROTECTION -> +5V_ALIM
- C25 pad 2: GND -> GND_ALIM
- C26 pad 1: VIN_PROTECTION -> +5V_ALIM
- C26 pad 2: GND -> GND_ALIM
- FB1 pad 2: VIN_PROTECTION -> +5V
- J14 pad 1: Net-(J14-3V3-Pad1) -> +3V3
- J14 pad 10: unconnected-(J14-GPIO15/UART_RXD-Pad10) -> /MCU/GPIO0
- J14 pad 14: Net-(J14-GND-Pad14) -> GND
- J14 pad 17: Net-(J14-3V3-Pad1) -> +3V3
- J14 pad 2: Net-(J14-5V-Pad2) -> +5V
- J14 pad 20: Net-(J14-GND-Pad14) -> GND
- J14 pad 25: Net-(J14-GND-Pad14) -> GND
- J14 pad 30: Net-(J14-GND-Pad14) -> GND
- J14 pad 34: Net-(J14-GND-Pad14) -> GND
- J14 pad 39: Net-(J14-GND-Pad14) -> GND
- J14 pad 4: Net-(J14-5V-Pad2) -> +5V
- J14 pad 6: Net-(J14-GND-Pad14) -> GND
- J14 pad 8: unconnected-(J14-GPIO14/UART_TXD-Pad8) -> /MCU/GPIO1
- J14 pad 9: Net-(J14-GND-Pad14) -> GND
- L2 pad 2: VIN_PROTECTION -> +5V_ALIM
- M1 pad 1: /Steppers/STEP1.13_2A -> Net-(J17-B)
- M1 pad 2: /Steppers/STEP1.14_2B -> Net-(J17-A)
- M1 pad 3: /Steppers/STEP1.12_1A -> Net-(J17-C)
- M1 pad 4: /Steppers/STEP1.11_1B -> Net-(J17-D)
- M2 pad 1: /Steppers/STEP2.13_2A -> Net-(J18-B)
- M2 pad 2: /Steppers/STEP2.14_2B -> Net-(J18-A)
- M2 pad 3: /Steppers/STEP2.12_1A -> Net-(J18-C)
- M2 pad 4: /Steppers/STEP2.11_1B -> Net-(J18-D)
- M3 pad 1: /Steppers/STEP3.13_2A -> Net-(J20-B)
- M3 pad 2: /Steppers/STEP3.14_2B -> Net-(J20-A)
- M3 pad 3: /Steppers/STEP3.12_1A -> Net-(J20-C)
- M3 pad 4: /Steppers/STEP3.11_1B -> Net-(J20-D)
- M4 pad 1: /Steppers/STEP6.13_2A -> Net-(J22-B)
- M4 pad 2: /Steppers/STEP6.14_2B -> Net-(J22-A)
- M4 pad 3: /Steppers/STEP6.12_1A -> Net-(J22-C)
- M4 pad 4: /Steppers/STEP6.11_1B -> Net-(J22-D)
- M5 pad 1: /Steppers/STEP5.13_2A -> Net-(J25-B)
- M5 pad 2: /Steppers/STEP5.14_2B -> Net-(J25-A)
- M5 pad 3: /Steppers/STEP5.12_1A -> Net-(J25-C)
- M5 pad 4: /Steppers/STEP5.11_1B -> Net-(J25-D)
- M6 pad 1: /Steppers/STEP4.13_2A -> Net-(J26-B)
- M6 pad 2: /Steppers/STEP4.14_2B -> Net-(J26-A)
- M6 pad 3: /Steppers/STEP4.12_1A -> Net-(J26-C)
- M6 pad 4: /Steppers/STEP4.11_1B -> Net-(J26-D)
- R10 pad 2: GND -> GND_ALIM
- R11 pad 1: Vcc_3V3 -> +3V3
- R12 pad 1: VIN_PROTECTION -> +5V_ALIM
- R13 pad 2: GND -> GND_ALIM
- R9 pad 1: +12V -> +12V_BAT
- TP1 pad 1: VIN_PROTECTION -> +5V
- TP2 pad 1: +12V -> +12V_BAT
- TP3 pad 1: Vcc_3V3 -> +3V3
- TP4 pad 1: VIN_PROTECTION -> +5V_ALIM
- TP5 pad 1: GND -> GND_ALIM
- U4 pad 1: VIN_PROTECTION -> +5V
- U4 pad 3: Vcc_3V3 -> +3V3
Other:
- board outline added: 100 x 92 mm
- copper layers 2 -> 4

Commit message: push pcb
Parts:
- added kibuzzard-67CE320A: G***, kibuzzard-67CE320A, B.Cu at (139.4, 82.2)
- added kibuzzard-67CE323D: G***, kibuzzard-67CE323D, B.Cu at (139.4, 110.9)
- added kibuzzard-67CE33A5: G***, kibuzzard-67CE33A5, B.Cu at (149.3, 57.0)
- added kibuzzard-67CE3450: G***, kibuzzard-67CE3450, B.Cu at (169.8, 57.0)
- added kibuzzard-67CE3465: G***, kibuzzard-67CE3465, B.Cu at (190.3, 57.0)
- added kibuzzard-67CE3487: G***, kibuzzard-67CE3487, B.Cu at (161.7, 136.0)
- added kibuzzard-67CE3498: G***, kibuzzard-67CE3498, B.Cu at (182.2, 136.0)
- added kibuzzard-67CE34A5: G***, kibuzzard-67CE34A5, B.Cu at (202.8, 136.0)
- moved M4 41.0 mm to (155.5, 139.8)
- moved M6 41.0 mm to (196.5, 139.9)
- turned R4 to 90 degrees
- renumbered TP2 to 12V, TP3 to 3v3, TP1 to 5V, TP4 to 5V, SW1 to BOOT, TP5 to GND, SW2 to RESET
Routing:
- net GND: track 0.00 -> 447.3 mm, vias 0 -> 56
- net +12V: track 0.00 -> 173.3 mm
- net +3V3: track 0.00 -> 154.1 mm, vias 0 -> 23
- net +5V: track 0.00 -> 151.6 mm, vias 0 -> 9
- net +12V_BAT: track 0.00 -> 90.5 mm, vias 0 -> 49
- net GND_ALIM: track 0.00 -> 81.8 mm, vias 0 -> 42
- net +3V3_I2C: track 0.00 -> 75.9 mm
- net GND_I2C: track 0.00 -> 63.6 mm, vias 0 -> 12
- net +5V_ALIM: track 0.00 -> 61.5 mm, vias 0 -> 76
- net /MCU/GPIO2: track 0.00 -> 57.2 mm, vias 0 -> 2
- net /MCU/GPIO3: track 0.00 -> 55.3 mm, vias 0 -> 2
- net /MCU/~{QSPI_CS_{0}}: track 0.00 -> 49.3 mm, vias 0 -> 3
- net /MCU/GPIO8: track 0.00 -> 48.0 mm, vias 0 -> 2
- net /MCU/GPIO5: track 0.00 -> 46.1 mm, vias 0 -> 2
- net /MCU/GPIO15: track 0.00 -> 45.1 mm, vias 0 -> 2
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- added copper zone on In2.Cu, net +12V_BAT
- added copper zone on In2.Cu, net +3V3
- added copper zone on In2.Cu, net +3V3_I2C
- added copper zone on In1.Cu, net +5V
- added copper zone on In2.Cu, net +5V_ALIM
- added copper zone on B.Cu, net GND
- added copper zone on F.Cu, net GND
- added copper zone on In1.Cu, net GND
- added copper zone on B.Cu, net GND_ALIM
- added copper zone on F.Cu, net GND_ALIM
- added copper zone on B.Cu, net GND_I2C
- added copper zone on F.Cu, net GND_I2C
Other:
- board text added: "12V"
- board text added: "3V3 SDA SCL GND"
- board text added: "5V 3V3 5V X"
- board text added: "Battery here!"
- board text added: "Fait par: Jacob Turcotte"
- board text added: "GND"
