File: Electric/Aeris control electrical plans/Cerbrum_Aeris/MCU.kicad_sch (KiCad schematic)
At the start: 34 parts, among them J1 USB_C_PICO, SW1 SW_BOOTSEL, SW2 SW_RESET, U1 SRV05-4, U2 RP2350B-QFN80, U3 W25Q128JVPIQ, Y1 CM4012M00012001

Commit message: push éelectrique pcb
Parts:
- L1: footprint (none) -> Resistor_SMD:R_0805_2012Metric
Other:
- note added: "I2C_0"
- note added: "I2C_1"
- note added: "M_Conn_LEFT"
- note added: "M_Conn_RIGHT"
- note added: "UART"
- note added: "Unused"
Changed lines of the file:
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@@
 		)
 	)
+	(text "M_Conn_LEFT"
+		(exclude_from_sim no)
+		(at 338.836 74.168 0)
+		(effects
+			(font
+				(size 1.27 1.27)
+				(thickness 0.254)
+				(bold yes)
+			)
+		)
+	)
 	(text "24"
 		(exclude_from_sim no)
@@
 		)
 	)
+	(text "Unused"
+		(exclude_from_sim no)
+		(at 337.312 127.254 0)
+		(effects
+			(font
+				(size 1.27 1.27)
+				(thickness 0.254)
+				(bold yes)
+			)
+		)
+	)
+	(text "I2C_0"
+		(exclude_from_sim no)
+		(at 334.518 55.118 0)
+		(effects
+			(font
+				(size 1.27 1.27)
+				(thickness 0.254)
+				(bold yes)
+			)
+		)
+	)
+	(text "M_Conn_RIGHT"
+		(exclude_from_sim no)
+		(at 340.868 97.282 0)
+		(effects
+			(font
+				(size 1.27 1.27)
+				(thickness 0.254)
+				(bold yes)
+			)
+		)
+	)
 	(text "12MHz"
 		(exclude_from_sim no)
@@
 		)
 	)
+	(text "I2C_1"
+		(exclude_from_sim no)
+		(at 334.518 60.198 0)
+		(effects
+			(font
+				(size 1.27 1.27)
+				(thickness 0.254)
+				(bold yes)
+			)
+		)
+	)
+	(text "UART"
+		(exclude_from_sim no)
+		(at 334.264 50.038 0)
+		(effects
+			(font
+				(size 1.27 1.27)
+				(thickness 0.254)
+				(bold yes)
+			)
+		)
+	)
 	(text "ADC"
 		(exclude_from_sim no)
@@
 	)
 	(bus_entry
+		(at 317.5 53.34)
+		(size 2.54 2.54)
+		(stroke
+			(width 0)
+			(type default)
+		)
+	)
+	(bus_entry
 		(at 317.5 45.72)
 		(size 2.54 2.54)
@@
 	)
 	(bus_entry
-		(at 317.5 53.34)
-		(size 2.54 2.54)
-		(stroke
-			(width 0)
-			(type default)
-		)
-	)
-	(bus_entry
 		(at 317.5 101.6)
 		(size 2.54 2.54)
@@
 		)
 	)
+	(bus
+		(pts
+			(xy 320.04 53.34) (xy 320.04 55.88)
+		)
+		(stroke
+			(width 0)
+			(type default)
+		)
+	)
 	(wire
 		(pts
@@
 		)
 	)
-	(bus
-		(pts
-			(xy 320.04 50.8) (xy 320.04 53.34)
-		)
-		(stroke
-			(width 0)
-			(type default)
-		)
-	)
 	(wire
 		(pts
@@
 		)
 	)
-	(bus
-		(pts
-			(xy 320.04 55.88) (xy 320.04 58.42)
-		)
-		(stroke
-			(width 0)
-			(type default)
-		)
-	)
 	(wire
 		(pts
@@
 		)
 	)
-	(hierarchical_label "GPIO[3..5]"
+	(hierarchical_label "GPIO[4..5]"
 		(shape input)
-		(at 320.04 58.1393 0)
+		(at 320.04 59.69 0)
+		(effects
+			(font
+				(size 1.27 1.27)
+			)
+			(justify left)
+		)
+	)
+	(hierarchical_label "GPIO[2..3]"
+		(shape input)
+		(at 320.04 54.61 0)
 		(effects
 			(font
@@
 		)
 	)
-	(hierarchical_label "GPIO[0..2]"
+	(hierarchical_label "GPIO[0..1]"
 		(shape input)
-		(at 320.04 50.8 0)
+		(at 320.04 49.53 0)
 		(effects
 			(font
@@
 			)
 		)
-		(property "Footprint" ""
+		(property "Footprint" "Resistor_SMD:R_0805_2012Metric"
 			(at 217.17 30.48 0)
 			(effects

Commit message: push kicad erreurs
Other:
- note added: "100k pas nécessaire"
- note added: "D+ et D- sont inversé"
- note added: "Maybe descendre à 1kOhm?"
- note added: "Pas 10µF Supposé être 4µ7F"
- note added: "Pull-up de 100k est pas nécessaire maybe 1k en série"
- note added: "X"
- note added: "^--Aucune différence"
- note added: "je vais changer la clock par celle recommandé par RPi..."
- note added: "maybe 1k en série avec xout"
Changed lines of the file:
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@@
+		)
+	)
+	(text "100k pas nécessaire"
+		(exclude_from_sim no)
+		(at 353.568 32.258 0)
+		(effects
+			(font
+				(size 1.27 1.27)
+				(color 255 5 0 1)
+			)
+		)
+	)
+	(text "Maybe descendre à 1kOhm?"
+		(exclude_from_sim no)
+		(at 195.072 60.198 0)
+		(effects
+			(font
+				(size 1.27 1.27)
+				(color 255 5 0 1)
+			)
 		)
 	)
@@
 		)
 	)
+	(text "^--Aucune différence"
+		(exclude_from_sim no)
+		(at 147.32 90.424 0)
+		(effects
+			(font
+				(size 1.27 1.27)
+				(thickness 0.1588)
+			)
+		)
+	)
 	(text "24"
 		(exclude_from_sim no)
@@
 		)
 	)
+	(text "X"
+		(exclude_from_sim no)
+		(at 357.378 32.258 0)
+		(effects
+			(font
+				(size 3 3)
+				(thickness 0.6)
+				(bold yes)
+				(italic yes)
+				(color 0 255 11 1)
+			)
+		)
+	)
 	(text "41"
 		(exclude_from_sim no)
@@
 		)
 	)
+	(text "je vais changer la clock par celle recommandé par RPi..."
+		(exclude_from_sim no)
+		(at 195.072 84.074 0)
+		(effects
+			(font
+				(size 1.27 1.27)
+				(thickness 0.254)
+				(bold yes)
+				(italic yes)
+			)
+		)
+	)
 	(text "ADC"
 		(exclude_from_sim no)
@@
 		)
 	)
+	(text "X"
+		(exclude_from_sim no)
+		(at 214.63 77.47 0)
+		(effects
+			(font
+				(size 3 3)
+				(thickness 0.6)
+				(bold yes)
+				(italic yes)
+				(color 0 255 11 1)
+			)
+		)
+	)
 	(text "51"
 		(exclude_from_sim no)
@@
 		)
 	)
+	(text "X"
+		(exclude_from_sim no)
+		(at 195.326 60.96 0)
+		(effects
+			(font
+				(size 3 3)
+				(thickness 0.6)
+				(bold yes)
+				(italic yes)
+				(color 0 255 11 1)
+			)
+		)
+	)
 	(text "32"
 		(exclude_from_sim no)
@@
 		)
 	)
+	(text "D+ et D- sont inversé\n"
+		(exclude_from_sim no)
+		(at 304.292 30.226 0)
+		(effects
+			(font
+				(size 1.27 1.27)
+				(color 255 5 0 1)
+			)
+		)
+	)
 	(text "ADC"
 		(exclude_from_sim no)
@@
 		)
 	)
+	(text "X"
+		(exclude_from_sim no)
+		(at 303.784 29.972 0)
+		(effects
+			(font
+				(size 3 3)
+				(thickness 0.6)
+				(bold yes)
+				(italic yes)
+				(color 0 255 11 1)
+			)
+		)
+	)
+	(text "Pull-up de 100k est pas nécessaire\nmaybe 1k en série"
+		(exclude_from_sim no)
+		(at 199.644 102.616 0)
+		(effects
+			(font
+				(size 1.27 1.27)
+				(color 255 5 0 1)
+			)
+		)
+	)
 	(text "I2C_1"
 		(exclude_from_sim no)
@@
 		)
 	)
+	(text "maybe 1k en série \navec xout"
+		(exclude_from_sim no)
+		(at 215.392 76.708 0)
+		(effects
+			(font
+				(size 1.27 1.27)
+				(color 255 5 0 1)
+			)
+		)
+	)
+	(text "Pas 10µF\nSupposé être 4µ7F\n"
+		(exclude_from_sim no)
+		(at 142.494 86.614 0)
+		(effects
+			(font
+				(size 1.27 1.27)
+				(color 255 5 0 1)
+			)
+		)
+	)
+	(text "X"
+		(exclude_from_sim no)
+		(at 195.834 101.346 0)
+		(effects
+			(font
+				(size 3 3)
+				(thickness 0.6)
+				(bold yes)
+				(italic yes)
+				(color 0 255 11 1)
+			)
+		)
+	)
